File: RC6502 ATTiny Clock/ATTiny Clock.sch (KiCad schematic (older format))
At the start: 9 parts, among them J1 CONN_01X39, J3 CONN_01X06, U1 ATTINY85-20PU, Y1 20Mhz

Commit message: Changed crystal footprint
Parts:
- Y1: footprint Crystals:Crystal_HC52-6mm_Vertical -> Crystals:Crystal_HC49-4H_Vertical
Changed lines of the file:
@@
 F 0 "Y1" H 2150 2750 50  0000 C CNN
 F 1 "20Mhz" H 2150 2450 50  0000 C CNN
-F 2 "Crystals:Crystal_HC52-6mm_Vertical" H 2150 2600 50  0001 C CNN
+F 2 "Crystals:Crystal_HC49-4H_Vertical" H 2150 2600 50  0001 C CNN
 F 3 "" H 2150 2600 50  0001 C CNN
 	1    2150 2600
