File: RC6502 General Video Adapter/RC6502 General Video Adapter.sch (KiCad schematic (older format))
At the start: 67 parts, among them U1 4040, U10 CY7C199, U11 74LS373, U12 74LS373, U13 74LS373, U14 74LS86, U15 74LS32, U16 74LS00, U17 74LS04, U2 4040, U3 74LS04, U4 74LS08, U5 74LS08, U6 74LS86, U7 74LS04, U9 74LS165

Commit message: Yeah, I'm not going to get this within 10x10cm :-(
Parts:
- removed U1, U2: 4040, symbol 4040
- removed U3: 74LS04, symbol 74LS04
- added C10, C11, C12, C13, C14, C15, C16, C17, C3, C4, C5, C6, C7, C8, C9: 100nF, Capacitors_THT:C_Disc_D4.7mm_W2.5mm_P5.00mm, symbol C_Small
- added U1, U2: 4040_vcc, Housings_DIP:DIP-16_W7.62mm_Socket, symbol 4040_vcc
- D1, D10, D11, D12, D13, D14, D15, D16, D2, D3, D4, D5, D6, D7, D8, D9: renamed from D?; footprint (none) -> Diodes_THT:D_DO-35_SOD27_P7.62mm_Horizontal
- R1, R10, R11, R12, R13, R14, R15, R16, R17, R18, R19, R2, R20, R3, R4, R5, R6, R7, R8, R9: renamed from R?; footprint (none) -> Resistors_THT:R_Axial_DIN0207_L6.3mm_D2.5mm_P10.16mm_Horizontal
- RV1: renamed from RV?; value POT -> 5k; footprint (none) -> Potentiometers:Potentiometer_Trimmer_Bourns_3296W
- RV2: renamed from RV?; footprint (none) -> Potentiometers:Potentiometer_Trimmer_Bourns_3296W
- U10: footprint (none) -> Housings_DIP:DIP-28_W7.62mm_Socket
- U11, U12, U13: value 74LS373 -> 74HCT373; footprint (none) -> Housings_DIP:DIP-20_W7.62mm_Socket
- U14, U6: value 74LS86 -> 74HCT86; footprint (none) -> Housings_DIP:DIP-14_W7.62mm_Socket
- U15: value 74LS32 -> 74HCT32; footprint (none) -> Housings_DIP:DIP-14_W7.62mm_Socket
- U15: renamed from U?; value 74LS32 -> 74HCT32; footprint (none) -> Housings_DIP:DIP-14_W7.62mm_Socket
- U16: value 74LS00 -> 74HCT00; footprint (none) -> Housings_DIP:DIP-14_W7.62mm_Socket
- U17, U3, U7: value 74LS04 -> 74HCT04; footprint (none) -> Housings_DIP:DIP-14_W7.62mm_Socket
- U4, U5: value 74LS08 -> 74HCT08; footprint (none) -> Housings_DIP:DIP-14_W7.62mm_Socket
- U9: value 74LS165 -> 74HCT165; footprint (none) -> Housings_DIP:DIP-16_W7.62mm_Socket
- Y1: renamed from Y?; footprint (none) -> Crystals:Crystal_HC49-4H_Vertical
- gave numbers to parts that had none: 7
Connections:
- net CLOCK: now also U1.10 (CLK)
- net GND: now also U14.10 (IN2), U14.4 (IN1), U14.5 (IN2), U14.9 (IN1), U15.10, U15.12, U15.13, U15.4, U15.5, U15.9, U17.3, C10.1, C11.1, C12.1, C13.1, C14.1, C15.1, C16.1, C17.1, C3.1, C4.1, C5.1, C6.1, C7.1, C8.1, C9.1, U1.8 (GND), U2.8 (GND)
- net N0: now also U1.9 (Q0)
- net N1: now also U1.7 (Q1)
- net N10: now also U1.15 (Q10)
- net N11: now also U1.1 (Q11), U2.10 (CLK)
- net N12: now also U2.9 (Q0)
- net N13: now also U2.7 (Q1)
- net N14: now also U2.6 (Q2)
- net N15: now also U2.5 (Q3)
- net N16: now also U2.3 (Q4)
- net N17: now also U2.2 (Q5)
- net N2: now also U1.6 (Q2)
- net N3: now also U1.5 (Q3)
- net N4: now also U1.3 (Q4)
- net N5: now also U1.2 (Q5)
- net N6: now also U1.4 (Q6)
- net N7: now also U1.13 (Q7)
- net N8: now also U1.12 (Q8)
- net N9: now also U1.14 (Q9)
- net RESET: now also U1.11 (Reset), U2.11 (Reset)
- net VCC: now also C10.2, C11.2, C12.2, C13.2, C14.2, C15.2, C16.2, C17.2, C3.2, C4.2, C5.2, C6.2, C7.2, C8.2, C9.2, U1.16 (VCC), U2.16 (VCC)
- no-connect marks 54 -> 62
Other:
- note added: "RC6502 General Video Adapter"
- note added: "Schematic based on MC3 Bitmapped Video Interface by Daniel Tufvesson\n(http://www.waveguide.se/?article=bitmapped-video-interface). Pin connector on the\nbottom of the PCB for use with RC6502 or RC2014 computer."
- moved on the sheet: C1, C2, U14B, U14C, U15B, U17B
