File: RC6502 VDU/RC6502 VDU.sch (KiCad schematic (older format))
At the start: 39 parts, among them J1 RC6502_Backplane, J2 VDU_BASE, J3 VIDEO, J4 Hole, J5 Hole, J6 Hole, J7 Hole, J8 RCA_PLUG, Q1 PN2222A, Q2 PN2222A, U1 MC6847, U10 74HCT00, U2 HM62256BLP-7, U3 74LS244, U4 74LS244, U5 74LS245, U6 74LS374, U7 74HCT138, U8 74HCT04, U9 74HCT00, X1 3.579545 MHz

Commit message: Changed VDU CS logic ins schematic
Parts:
- removed Q1, Q2: PN2222A, TO_SOT_Packages_THT:TO-92_Molded_Narrow, symbol PN2222A
- removed R1, R2, R5: 1k, Resistors_THT:R_Axial_DIN0207_L6.3mm_D2.5mm_P5.08mm_Vertical, symbol R
- removed R3: 180, Resistors_THT:R_Axial_DIN0207_L6.3mm_D2.5mm_P5.08mm_Vertical, symbol R
- removed R4: 6.2k, Resistors_THT:R_Axial_DIN0207_L6.3mm_D2.5mm_P5.08mm_Vertical, symbol R
- removed U10, U9: 74HCT00, Housings_DIP:DIP-14_W7.62mm, symbol 74HCT00
- removed U8: 74HCT04, Housings_DIP:DIP-14_W7.62mm, symbol 74LS04
- added C12: 100nF, Capacitors_THT:C_Disc_D4.7mm_W2.5mm_P5.00mm, symbol C
- added U10: 74LS02, symbol 74LS02
- added U11: VDU_Port, vdu_amplifier:VDU Module, symbol VDU_Port
- added U12: 74LS374, Housings_DIP:DIP-20_W7.62mm, symbol 74LS374
- added U8: 74LS32, symbol 74LS32
- added U9: 74HCT138, Housings_DIP:DIP-16_W7.62mm_Socket, symbol 74LS138
- J2: footprint Pin_Headers:Pin_Header_Straight_1x10_Pitch2.54mm -> Pin_Headers:Pin_Header_Straight_2x05_Pitch2.54mm
- J3: footprint Pin_Headers:Pin_Header_Straight_1x05_Pitch2.54mm -> Pin_Headers:Pin_Header_Straight_1x07_Pitch2.54mm; symbol Conn_01x05 -> Conn_01x07
Connections:
- net A10: now also U9.1 (A0)
- net A11: now also U12.3 (D0), U9.2 (A1); no longer U3.8 (I3a)
- net A12: now also U12.4 (D1); no longer U3.11 (I0b)
- net A13: no longer U3.13 (I1b)
- net A14: no longer U3.15 (I2b)
- net A15: no longer U3.17 (I3b)
- net GND: now also J3.6 (Pin_6), U3.11 (I0b), U3.13 (I1b), U3.15 (I2b), U3.17 (I3b), U3.8 (I3a), C12.2, U10.11, U10.12, U10.7 (GND), U10.7 (GND), U10.7 (GND), U10.7 (GND), U11.6 (GND), U12.10 (GND), U12.13 (D4), U12.14 (D5), U12.17 (D6), U12.18 (D7), U12.7 (D2), U12.8 (D3), U8.1, U8.10, U8.2, U8.4, U8.5, U8.7 (GND), U8.7 (GND), U8.7 (GND), U8.7 (GND), U8.9, U9.4 (E1), U9.8 (GND)
- net PHI2: now also U9.6 (E3)
- net R/~W: now also U5.1 (A->B), U8.13, U9.3 (A2)
- net RAM_RW: now also U8.11; no longer U5.1 (A->B)
- net VA11: now also U12.2 (O0); no longer U3.12 (O3a)
- net VA12: now also U12.5 (O1); no longer U3.9 (O0b)
- net VA13: no longer U3.7 (O1b)
- net VA14: no longer U3.5 (O2b)
- net VCC: now also J3.7 (Pin_7), C12.1, U10.14 (VCC), U10.14 (VCC), U10.14 (VCC), U10.14 (VCC), U11.1 (VCC), U12.20 (VCC), U8.14 (VCC), U8.14 (VCC), U8.14 (VCC), U8.14 (VCC), U9.16 (VCC)
- net VDU_BASE: now also U9.5 (E2)
- net Y: now also U11.2 (VID_IN)
- net ~CS_RAM_EXT: now also U10.10, U12.1 (OE), U8.12
- net at J8.2 (In): now also U11.3 (VID_OUT)
- net ~CS_CTRL_EXT renamed ~REG0
- net ~REG0: now also U9.13 (O2)
- new net: U10.6, U9.10 (O5)
- new net: U10.5, U9.11 (O4)
- new net: U10.3, U9.14 (O1)
- new net: U10.2, U9.15 (O0)
- new net: U10.1, U10.8
- new net: U10.4, U10.9
- new net ~REG1: U12.11 (Cp), U9.12 (O3)
- no-connect marks 13 -> 30
Other:
- moved on the sheet: C1, C10, C2, C3, C4, C5, C6, C7, C8, C9, J4, J5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

Commit message: Assigned new footprints
Parts:
- U10, U8: footprint (none) -> Housings_DIP:DIP-14_W7.62mm_Socket
- X1: footprint Oscillators:Oscillator_DIP-14 -> Oscillator:Oscillator_DIP-14
Changed lines of the file:
@@
 F 0 "X1" H 2500 2725 50  0000 L CNN
 F 1 "3.579545 MHz" H 2750 2225 50  0000 L CNN
-F 2 "Oscillators:Oscillator_DIP-14" H 3150 2125 50  0001 C CNN
+F 2 "Oscillator:Oscillator_DIP-14" H 3150 2125 50  0001 C CNN
 F 3 "" H 2600 2475 50  0001 C CNN
 	1    2700 2475
@@
 F 0 "U10" H 3300 3800 50  0000 C CNN
 F 1 "74LS02" H 3350 3700 50  0000 C CNN
-F 2 "" H 3300 3750 50  0001 C CNN
+F 2 "Housings_DIP:DIP-14_W7.62mm_Socket" H 3300 3750 50  0001 C CNN
 F 3 "" H 3300 3750 50  0001 C CNN
 	1    3300 3750
@@
 F 0 "U10" H 3300 4300 50  0000 C CNN
 F 1 "74LS02" H 3350 4200 50  0000 C CNN
-F 2 "" H 3300 4250 50  0001 C CNN
+F 2 "Housings_DIP:DIP-14_W7.62mm_Socket" H 3300 4250 50  0001 C CNN
 F 3 "" H 3300 4250 50  0001 C CNN
 	2    3300 4250
@@
 F 0 "U10" H 4650 4050 50  0000 C CNN
 F 1 "74LS02" H 4700 3950 50  0000 C CNN
-F 2 "" H 4650 4000 50  0001 C CNN
+F 2 "Housings_DIP:DIP-14_W7.62mm_Socket" H 4650 4000 50  0001 C CNN
 F 3 "" H 4650 4000 50  0001 C CNN
 	3    4650 4000
@@
 F 0 "U10" H 6275 5975 50  0000 C CNN
 F 1 "74LS02" H 6325 5875 50  0000 C CNN
-F 2 "" H 6275 5925 50  0001 C CNN
+F 2 "Housings_DIP:DIP-14_W7.62mm_Socket" H 6275 5925 50  0001 C CNN
 F 3 "" H 6275 5925 50  0001 C CNN
 	4    6275 5925
@@
 F 0 "U8" H 6000 4400 50  0000 C CNN
 F 1 "74LS32" H 6000 4300 50  0000 C CNN
-F 2 "" H 6000 4350 50  0001 C CNN
+F 2 "Housings_DIP:DIP-14_W7.62mm_Socket" H 6000 4350 50  0001 C CNN
 F 3 "" H 6000 4350 50  0001 C CNN
 	4    6000 4350
@@
 F 0 "U8" H 4850 5975 50  0000 C CNN
 F 1 "74LS32" H 4850 5875 50  0000 C CNN
-F 2 "" H 4850 5925 50  0001 C CNN
+F 2 "Housings_DIP:DIP-14_W7.62mm_Socket" H 4850 5925 50  0001 C CNN
 F 3 "" H 4850 5925 50  0001 C CNN
 	1    4850 5925
@@
 F 0 "U8" H 5325 5975 50  0000 C CNN
 F 1 "74LS32" H 5325 5875 50  0000 C CNN
-F 2 "" H 5325 5925 50  0001 C CNN
+F 2 "Housings_DIP:DIP-14_W7.62mm_Socket" H 5325 5925 50  0001 C CNN
 F 3 "" H 5325 5925 50  0001 C CNN
 	2    5325 5925
@@
 F 0 "U8" H 5800 5975 50  0000 C CNN
 F 1 "74LS32" H 5800 5875 50  0000 C CNN
-F 2 "" H 5800 5925 50  0001 C CNN
+F 2 "Housings_DIP:DIP-14_W7.62mm_Socket" H 5800 5925 50  0001 C CNN
 F 3 "" H 5800 5925 50  0001 C CNN
 	3    5800 5925
