File: RC6502 RIOT/RC6502 RIOT.sch (KiCad schematic (older format))
At the start: 25 parts, among them J1 LEFT PLAYER, J2 VDU_BASE, J3 Analog, J4 RIGHT PLAYER, J5 AUX, J9 RC6502_Backplane_Extra, SW1 SELECT, SW2 START, U1 RIOT, U2 74HCT138

Commit message: RIOT module layout done
Parts:
- added JP11: RAM_EN, Pin_Headers:Pin_Header_Straight_1x03_Pitch2.54mm, symbol Jumper_NC_Dual
- J1, J4: footprint (none) -> RND_DSUB:DSUB-9_Male_Vertical_Pitch2.77x2.84mm
- J3: footprint (none) -> Pin_Headers:Pin_Header_Straight_1x04_Pitch2.54mm
- J5, JP10, JP8, JP9: footprint (none) -> Pin_Headers:Pin_Header_Straight_1x03_Pitch2.54mm
- JP6: value RS_SEL -> RAM_SEL
- R1: footprint (none) -> Resistors_THT:R_Axial_DIN0207_L6.3mm_D2.5mm_P10.16mm_Horizontal
- SW1, SW2: footprint (none) -> Buttons_Switches_THT:SW_PUSH_6mm
- U1: footprint (none) -> Housings_DIP:DIP-40_W15.24mm_Socket
Connections:
- net VCC: now also JP11.1
- net ~RS: now also JP11.2; no longer JP6.2
- net at R1.2: now also JP1.1; no longer JP1.3
- net at JP7.2: now also JP1.3; no longer JP1.1
- new net: JP11.3, JP6.2
Other:
- note added: "RC6502 RIOT 2600"
- note added: "RIOT card for the RC6502 computer, modelled after the input side of the Atari 2600 -\ntherefore features the same switches and joystick ports. Addressing can be jumpered to\nAtari 2600-mode, when doing so it assumes the presence of the corresponding\nTIA-module."
- note removed: "RC6502 RIOT"
- note removed: "RIOT card for the RC6502 computer, modelled after the input side of the Atari 2600 -\ntherefore features the same switches and joystick ports. Adressing can be jumpered to\nAtari 2600-mode, when doing so it assumes the presence of the corresponding\nTIA-module."
Changed lines of the file:
@@
 Comment4 ""
 $EndDescr
-Text Notes 7975 7500 2    60   ~ 0
-RC6502 RIOT
+Text Notes 7350 7500 0    60   ~ 0
+RC6502 RIOT 2600
 Text Notes 10650 7650 2    60   ~ 0
 A
@@
 	8375 1825 9025 1825
 Wire Bus Line
-	9600 6200 9600 525
+	9600 525  9600 6200
 Wire Wire Line
 	5225 2025 5650 2025
@@
 F 0 "U1" H 6300 2275 60  0000 C CNN
 F 1 "RIOT" V 6300 1925 60  0000 C CNN
-F 2 "" H 5800 2225 60  0000 C CNN
+F 2 "Housings_DIP:DIP-40_W15.24mm_Socket" H 5800 2225 60  0001 C CNN
 F 3 "" H 5800 2225 60  0000 C CNN
 	1    6300 2025
@@
 F 0 "R1" V 8755 3825 50  0000 C CNN
 F 1 "3k3" V 8675 3825 50  0000 C CNN
-F 2 "" V 8605 3825 50  0001 C CNN
+F 2 "Resistors_THT:R_Axial_DIN0207_L6.3mm_D2.5mm_P10.16mm_Horizontal" V 8605 3825 50  0001 C CNN
 F 3 "" H 8675 3825 50  0001 C CNN
 	1    8675 3825
@@
 F 3 "" H 8675 4225 50  0001 C CNN
 	1    8675 4225
-	0    -1   -1   0
+	0    -1   1    0
 $EndComp
 Wire Wire Line
@@
 Wire Wire Line
 	8675 4475 8675 4875
-$Comp
-L Jumper_NC_Dual JP6
-U 1 1 5C64A264
-P 8800 2725
-F 0 "JP6" H 8850 2625 50  0000 L CNN
-F 1 "RS_SEL" H 8800 2825 50  0000 C BNN
-F 2 "Pin_Headers:Pin_Header_Straight_1x03_Pitch2.54mm" H 8800 2725 50  0001 C CNN
-F 3 "" H 8800 2725 50  0001 C CNN
-	1    8800 2725
-	0    1    1    0
-$EndComp
 Entry Wire Line
 	9500 2400 9600 2500
-Wire Wire Line
-	8800 2400 9500 2400
-Wire Wire Line
-	8800 2475 8800 2400
 Text Label 8400 2725 0    60   ~ 0
 ~RS
 Entry Wire Line
 	8375 2725 8275 2625
-Wire Wire Line
-	8375 2725 8700 2725
 Wire Notes Line
 	8125 3475 9375 3475
@@
 Wire Wire Line
 	8800 1325 9125 1325
-Wire Wire Line
-	8800 3050 9500 3050
-Wire Wire Line
-	8800 3050 8800 2975
 Entry Wire Line
 	9500 3050 9600 3150
@@
 F 0 "J4" H 6975 5575 50  0000 C CNN
 F 1 "RIGHT PLAYER" H 6975 4450 50  0000 C CNN
-F 2 "" H 6975 5025 50  0001 C CNN
+F 2 "RND_DSUB:DSUB-9_Male_Vertical_Pitch2.77x2.84mm" H 6975 5025 50  0001 C CNN
 F 3 "" H 6975 5025 50  0001 C CNN
 	1    6975 5025
@@
 F 0 "J1" H 5225 5575 50  0000 C CNN
 F 1 "LEFT PLAYER" H 5225 4450 50  0000 C CNN
-F 2 "" H 5225 5025 50  0001 C CNN
+F 2 "RND_DSUB:DSUB-9_Male_Vertical_Pitch2.77x2.84mm" H 5225 5025 50  0001 C CNN
 F 3 "" H 5225 5025 50  0001 C CNN
 	1    5225 5025
@@
 F 0 "J3" H 6875 4175 50  0000 C CNN
 F 1 "Analog" H 6875 3675 50  0000 C CNN
-F 2 "" H 6875 3975 50  0001 C CNN
+F 2 "Pin_Headers:Pin_Header_Straight_1x04_Pitch2.54mm" H 6875 3975 50  0001 C CNN
 F 3 "" H 6875 3975 50  0001 C CNN
 	1    6875 3975
@@
 	4400 5325 4500 5425
 Wire Bus Line
-	6150 6200 6150 3775
+	6150 3775 6150 6200
 Wire Bus Line
 	4400 4525 4400 6200
@@
 F 0 "JP8" H 3225 3775 50  0000 L CNN
 F 1 "B/W" H 3175 3975 50  0000 C BNN
-F 2 "" H 3175 3875 50  0001 C CNN
+F 2 "Pin_Headers:Pin_Header_Straight_1x03_Pitch2.54mm" H 3175 3875 50  0001 C CNN
 F 3 "" H 3175 3875 50  0001 C CNN
 	1    3175 3875
@@
 F 0 "JP9" H 3225 4550 50  0000 L CNN
 F 1 "L_DIFF" H 3175 4750 50  0000 C BNN
-F 2 "" H 3175 4650 50  0001 C CNN
+F 2 "Pin_Headers:Pin_Header_Straight_1x03_Pitch2.54mm" H 3175 4650 50  0001 C CNN
 F 3 "" H 3175 4650 50  0001 C CNN
 	1    3175 4650
@@
 F 0 "JP10" H 3225 5300 50  0000 L CNN
 F 1 "R_DIFF" H 3175 5500 50  0000 C BNN
-F 2 "" H 3175 5400 50  0001 C CNN
+F 2 "Pin_Headers:Pin_Header_Straight_1x03_Pitch2.54mm" H 3175 5400 50  0001 C CNN
 F 3 "" H 3175 5400 50  0001 C CNN
 	1    3175 5400
@@
 F 0 "SW1" H 1800 4050 50  0000 L CNN
 F 1 "SELECT" H 1750 3890 50  0000 C CNN
-F 2 "" H 1750 4150 50  0001 C CNN
+F 2 "Buttons_Switches_THT:SW_PUSH_6mm" H 1750 4150 50  0001 C CNN
 F 3 "" H 1750 4150 50  0001 C CNN
 	1    1750 3950
@@
 F 0 "SW2" H 1800 4825 50  0000 L CNN
 F 1 "START" H 1750 4665 50  0000 C CNN
-F 2 "" H 1750 4925 50  0001 C CNN
+F 2 "Buttons_Switches_THT:SW_PUSH_6mm" H 1750 4925 50  0001 C CNN
 F 3 "" H 1750 4925 50  0001 C CNN
 	1    1750 4725
@@
 F 0 "J5" H 1825 5800 50  0000 C CNN
 F 1 "AUX" H 1825 5400 50  0000 C CNN
-F 2 "" H 1825 5600 50  0001 C CNN
+F 2 "Pin_Headers:Pin_Header_Straight_1x03_Pitch2.54mm" H 1825 5600 50  0001 C CNN
 F 3 "" H 1825 5600 50  0001 C CNN
 	1    1825 5600
@@
 Input switches
 Text Notes 7025 6975 0    60   ~ 0
-RIOT card for the RC6502 computer, modelled after the input side of the Atari 2600 -\ntherefore features the same switches and joystick ports. Adressing can be jumpered to\nAtari 2600-mode, when doing so it assumes the presence of the corresponding\nTIA-module.
+RIOT card for the RC6502 computer, modelled after the input side of the Atari 2600 -\ntherefore features the same switches and joystick ports. Addressing can be jumpered to\nAtari 2600-mode, when doing so it assumes the presence of the corresponding\nTIA-module.
+$Comp
+L Jumper_NC_Dual JP6
+U 1 1 5C669D81
+P 9075 2725
+F 0 "JP6" H 9125 2625 50  0000 L CNN
+F 1 "RAM_SEL" H 9075 2825 50  0000 C BNN
+F 2 "Pin_Headers:Pin_Header_Straight_1x03_Pitch2.54mm" H 9075 2725 50  0001 C CNN
+F 3 "" H 9075 2725 50  0001 C CNN
+	1    9075 2725
+	0    1    1    0
+$EndComp
+Wire Wire Line
+	9075 2475 9075 2400
+Wire Wire Line
+	9075 2975 9075 3050
+Wire Wire Line
+	9075 3050 9500 3050
+Wire Wire Line
+	9075 2400 9500 2400
+$Comp
+L Jumper_NC_Dual JP11
+U 1 1 5C66BB42
+P 8700 2725
+F 0 "JP11" H 8750 2625 50  0000 L CNN
+F 1 "RAM_EN" H 8700 2825 50  0000 C BNN
+F 2 "Pin_Headers:Pin_Header_Straight_1x03_Pitch2.54mm" H 8700 2725 50  0001 C CNN
+F 3 "" H 8700 2725 50  0001 C CNN
+	1    8700 2725
+	0    1    1    0
+$EndComp
+Wire Wire Line
+	8375 2725 8600 2725
+Wire Wire Line
+	8975 2725 8900 2725
+Wire Wire Line
+	8900 2725 8900 3050
+Wire Wire Line
+	8900 3050 8700 3050
+Wire Wire Line
+	8700 3050 8700 2975
+$Comp
+L VCC #PWR021
+U 1 1 5C66C811
+P 8700 2475
+F 0 "#PWR021" H 8700 2325 50  0001 C CNN
+F 1 "VCC" H 8700 2625 50  0000 C CNN
+F 2 "" H 8700 2475 50  0001 C CNN
+F 3 "" H 8700 2475 50  0001 C CNN
+	1    8700 2475
+	1    0    0    -1
+$EndComp
 $EndSCHEMATC
