File: RC6502 Terminal/RC6502 Terminal.sch (KiCad schematic (older format))
At the start: 44 parts, among them J1 RC6502_Backplane, J2 KBD_SER, J3 VID_SER, J4 KBD_ICSP, J5 VID_ICSP, J6 AUDIO, J7 VIDEO, J8 Keyboard, SW1 KBD_RES, SW2 VID_RES, U1 MC6821, U2 74LS138, U3 74LS00, U4 ATMEGA328_MCU, U5 ATMEGA328_MCU, Y1 16Mhz, Y2 16Mhz

Commit message: Terminal silkscreen got striped
Parts:
- added JP3: SELECT, Pin_Headers:Pin_Header_Straight_1x03_Pitch2.54mm, symbol Jumper_NC_Dual
- J2, J3: footprint Pin_Headers:Pin_Header_Angled_1x06_Pitch2.54mm -> Pin_Headers:Pin_Header_Straight_1x06_Pitch2.54mm
- U4, U5: footprint Housings_DIP:DIP-28_W7.62mm_Socket_LongPads -> Housings_DIP:DIP-28_W7.62mm_Socket
Connections:
- net A4: now also U3.4, U3.5, JP3.1; no longer U1.22 (CS0)
- net GND: now also C1.2, C2.2, C3.2, D3.1 (K), D4.1 (K); no longer C1.1, C2.1, C3.1, R6.2, R7.2, U3.4, U3.5
- net PS2_CLK: now also R8.2; no longer R8.1
- net PS2_DATA: now also R9.2; no longer R9.1
- net VCC: now also C1.1, C2.1, C3.1; no longer C1.2, C2.2, C3.2
- net at C7.1, J2.4 (Pin_4), J4.2 (Pin_2)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: now also R8.1, R9.1, U4.20 (AVCC); no longer R8.2, R9.2
- net at C6.1, Y1.1: now also U4.9 (XTAL1); no longer U4.1 (~RESET)
- net at U4.10 (XTAL2): now also C10.1, Y1.2
- net at U4.16 ((PCINT2/OC1B/~SS~)PB2): now also R7.2; no longer D4.2 (A)
- net at C4.2, J4.5 (Pin_5), R1.1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: now also U4.1 (~RESET); no longer U4.20 (AVCC)
- net at C8.1, J3.4 (Pin_4), J5.2 (Pin_2)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: now also U5.20 (AVCC)
- net at C11.1, Y2.1: now also U5.9 (XTAL1); no longer U5.1 (~RESET)
- net at U5.10 (XTAL2): now also C12.1, Y2.2
- net at U5.16 ((PCINT2/OC1B/~SS~)PB2): now also R6.2; no longer D3.2 (A)
- net at C5.2, J5.5 (Pin_5), R2.1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: now also U5.1 (~RESET); no longer U5.20 (AVCC)
- net at D2.1 (K): now also R4.2; no longer R4.1
- net at D1.1 (K): now also R3.2; no longer R3.1
- net at J7.2 (In), R5.1: now also R3.1, R4.1; no longer R3.2, R4.2
- net at U3.6: now also JP3.3
- net at R6.1: now also D3.2 (A); no longer D3.1 (K)
- net at R7.1: now also D4.2 (A); no longer D4.1 (K)
- new net: JP3.2, U1.22 (CS0)
- no-connect marks 43 -> 42
Other:
- note added: "A"
- note added: "Address decoding places PIA at the expected addresses\n$D010 to $D012, these registers are mirrored across the\nentire $Dxxx range. SELECT should be on 1-2, 2-3 is used\nif this card should instead be placed on $D000 to $D002\n(for debugging)."
- moved on the sheet: C10, C11, C12, C6, D3, D4, J2, J3, R6, R7, U3B, U3D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
