File: RC6502 Terminal/RC6502 Terminal.kicad_pcb (KiCad board)
At the start: 2 copper layers, 99.1 x 81.9 mm, 44 parts, among them J1 RC6502_Backplane, J2 KBD_SER, J3 VID_SER, J4 KBD_ICSP, J5 VID_ICSP, J6 AUDIO, J7 VIDEO, J8 KEYBOARD, SW1 KBD_RES, SW2 VID_RES, U1 MC6821, U2 74LS138, U3 74LS00, U4 ATMEGA328_MCU, U5 ATMEGA328_MCU, Y1 16Mhz, Y2 16Mhz

Commit message: Terminal gerber export
Parts:
- added JP3: SELECT, Pin_Headers:Pin_Header_Straight_1x03_Pitch2.54mm, F.Cu at (177.8, 121.3)
- J8: value KEYBOARD -> Keyboard
Connections:
- U1 pad 22: /A4 -> Net-(JP3-Pad2)
- U3 pad 4: GND -> /A4
- U3 pad 5: GND -> /A4
- U3 pad 6: (no net) -> Net-(JP3-Pad3)
Routing:
- net Net-(JP3-Pad2): track 0.00 -> 93.4 mm, vias 0 -> 2
- net /A4: track 79.2 -> 33.0 mm, vias 0 -> 2
- net Net-(JP3-Pad3): track 0.00 -> 17.6 mm
Other:
- board text added: "GND"
- board text added: "RST"
- board text added: "RXD"
- board text added: "TXD"
- board text added: "VCC"
